File: schematic_files/ZetaBot.kicad_pcb (KiCad board)
At the start: 2 copper layers, 241.5 x 110.5 mm, 17 parts, among them J1 USB C PD Modulle, J2 Conn_01x05, J3 MOTOR_L, J4 MOTOR_R, SW1 SW_SPDT, U1 RPI5, U1 RPLIDAR C1, U2 Buck Converter

Commit message: Updated buck converter and re designed layout. Need to DRC.
Parts:
- U2: footprint deltabot:BUCK_CONV -> ZetaBotFootprints:BUCK_CONV
- moved C1 124.3 mm to (183.2, 51.0), turned to 0 degrees
- moved C2 94.7 mm to (184.4, 67.2), turned to 180 degrees
- moved F1 45.8 mm to (189.5, 127.0), turned to 90 degrees
- moved U2 29.5 mm to (158.0, 81.0), turned to 90 degrees
- moved C3 20.7 mm to (60.0, 114.4), turned to 90 degrees
- moved J2 17.9 mm to (58.5, 88.0)
- moved C6 17.9 mm to (58.7, 81.6)
- moved U1 17.9 mm to (106.0, 108.5)
- turned SW1 to 180 degrees
Routing:
- net +5V: track 339.6 -> 403.9 mm, vias 1 -> 2
- net Net-(SW1-B): track 70.4 -> 13.2 mm
- net PWM_L: track 282.8 -> 321.2 mm, vias 2 -> 1
- net +9V: track 62.9 -> 87.0 mm
- net PWM_R: track 116.5 -> 134.4 mm
- net Net-(J1-VCC): track 15.7 -> 21.2 mm
Other:
- outline, holes or cut-outs redrawn
