File: schematic_files/ZetaBot.kicad_pcb (KiCad board)
At the start: 2 copper layers, 241.5 x 110.5 mm, 23 parts, among them J1 USB C PD Modulle, J2 Conn_01x05, J3 MOTOR_L, J4 MOTOR_R, SW1 SW_SPDT, U1 RPI5, U1 RPLIDAR C1, U2 Buck Converter

Commit message: Updated the nets of the motors (L-R) and the pin headers.
Parts:
- J2: footprint ZetaBotFootprints:PinHeader_1x05_P2.54mm_Vertical -> Connector_PinHeader_2.54mm:PinHeader_1x05_P2.54mm_Vertical
- J3, J4: moved to B.Cu
- turned J3 to 180 degrees
- turned J4 to 0 degrees
Connections:
- J3 pad 1: PWM_L -> PWM_R
- J4 pad 1: PWM_R -> PWM_L
- U1 pad 12: PWM_L -> PWM_R
- U1 pad 35: PWM_R -> PWM_L
Routing:
- net PWM_L: track 314.0 -> 134.4 mm, vias 1 -> 0
- net PWM_R: track 134.4 -> 312.7 mm, vias 1 -> 0
- net +5V: track 402.4 -> 387.1 mm
