File: schematic_files/ZetaBot.kicad_sch (KiCad schematic)
At the start: 16 parts, among them J1 USB C PD Modulle, J2 Conn_01x05, J3 MOTOR_L, J4 MOTOR_R, SW1 SW_SPDT, U1 RPI5, U2 Buck Converter

Commit message: 2nd revision. DRC passed.
Other:
- company: (none) -> Bernd Porr
Changed lines of the file:
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@@
 	(title_block
 		(title "DeltaBot Schematic")
+		(date "2026-04-12")
+		(rev "2")
+		(company "Bernd Porr")
+		(comment 1 "GPL")
 	)
 	(rectangle

Commit message: Updated the nets of the motors (L-R) and the pin headers.
Connections:
- net PWM_L: now also J4.1 (Pin_1), U1.35 (GPIO19_PWM0/CHAN2); no longer J3.1 (Pin_1), U1.12 (GPIO18_PWM0/CHAN2)
- net PWM_R: now also J3.1 (Pin_1), U1.12 (GPIO18_PWM0/CHAN2); no longer J4.1 (Pin_1), U1.35 (GPIO19_PWM0/CHAN2)
Changed lines of the file:
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@@
 		)
 	)
-	(global_label "PWM_L"
+	(global_label "PWM_R"
 		(shape input)
 		(at 179.07 52.07 0)
@@
 		)
 	)
-	(global_label "PWM_L"
+	(global_label "PWM_R"
 		(shape input)
 		(at 68.58 116.84 180)
@@
 		)
 	)
-	(global_label "PWM_R"
+	(global_label "PWM_L"
 		(shape input)
 		(at 101.6 78.74 180)
@@
 		)
 	)
-	(global_label "PWM_R"
+	(global_label "PWM_L"
 		(shape input)
 		(at 68.58 92.71 180)
