File: hardware/ZetaBot.kicad_pcb (KiCad board)
At the start: 2 copper layers, 241.5 x 110.5 mm, 19 parts, among them J1 USB C PD Modulle, J2 Conn_01x05, J3 MOTOR_L, J4 MOTOR_R, SW1 SW_SPDT, U1 RPI5, U1 RPLIDAR C1, U2 Buck Converter

Commit message: Added header for Gyro and moved switch to post buck converter.
Parts:
- added J5: LSM6DSOX, Connector_PinHeader_2.54mm:PinHeader_1x05_P2.54mm_Vertical, F.Cu at (181.0, 90.1)
- moved SW1 89.6 mm to (216.0, 51.0), turned to 0 degrees
- moved F1 22.7 mm to (189.6, 106.0), turned to -90 degrees
- moved R1 16.0 mm to (187.5, 68.0)
- moved C2 3.20 mm to (184.5, 64.0), turned to 0 degrees
Connections:
- C1 pad 1: +5V -> Net-(SW1-B)
- C2 pad 1: +5V -> Net-(SW1-B)
- F1 pad 1: Net-(SW1-B) -> +9V
- R1 pad 1: +5V -> Net-(SW1-B)
- SW1 pad 1: +9V -> unconnected-(SW1-A-Pad1)
- SW1 pad 3: unconnected-(SW1-C-Pad3) -> +5V
- U1 pad 1: unconnected-(U1-3.3V-Pad1) -> Net-(J5-Pin_1)
- U1 pad 11: unconnected-(U1-GPIO17-Pad11) -> Net-(J5-Pin_5)
- U1 pad 3: unconnected-(U1-GPIO02_I2C1/SDA-Pad3) -> Net-(J5-Pin_3)
- U1 pad 5: unconnected-(U1-GPIO03_I2C1/SCL-Pad5) -> Net-(J5-Pin_4)
- U2 pad 3: +5V -> Net-(SW1-B)
Routing:
- net Net-(J5-Pin_1): track 0.00 -> 122.7 mm
- net Net-(J5-Pin_4): track 0.00 -> 122.0 mm
- net Net-(J5-Pin_3): track 0.00 -> 121.1 mm
- net Net-(J5-Pin_5): track 0.00 -> 118.6 mm
- net Net-(SW1-B): track 12.3 -> 101.9 mm
- net +5V: track 387.1 -> 343.2 mm, vias 2 -> 1
- net +9V: track 87.0 -> 46.1 mm
- net Net-(D1-A): track 6.27 -> 14.3 mm
- net Net-(F1-Pad2): track 27.0 -> 25.6 mm
- net PWM_R: track 312.7 -> 311.7 mm

Commit message: Moved switch out of the way of the servo
Parts:
- moved SW1 8.56 mm to (207.5, 52.0), turned to -90 degrees
- moved C1 2.26 mm to (186.5, 51.8), turned to 90 degrees
Routing:
- net Net-(SW1-B): track 101.9 -> 77.8 mm
- net +5V: track 343.2 -> 332.2 mm
Other:
- board text added: "Off"
- board text added: "On"
- board text removed: "OFF"
- board text removed: "ON"

Commit message: Now 99% of all tracks are on the top layer assuming we'll have vias!
Parts:
- J3: value MOTOR_L -> MOTOR_R
- J4: value MOTOR_R -> MOTOR_L
- moved J5 20.0 mm to (201.0, 89.9)
- moved SW1 5.70 mm to (201.8, 51.8)
- moved C2 4.20 mm to (184.6, 59.8)
- moved R1 0.93 mm to (187.8, 67.1)
- moved C3 0.15 mm to (60.0, 114.2)
Routing:
- net Net-(J5-Pin_5): track 118.6 -> 138.6 mm
- net Net-(J5-Pin_3): track 121.1 -> 140.7 mm
- net Net-(J5-Pin_1): track 122.7 -> 142.1 mm
- net Net-(J5-Pin_4): track 122.0 -> 141.1 mm
- net PWM_R: track 311.7 -> 316.3 mm
- net Net-(SW1-B): track 77.8 -> 73.3 mm
- net LIDAR_TX: track 30.0 -> 26.5 mm, vias 1 -> 0
- net Net-(D1-A): track 14.3 -> 16.2 mm
- net LIDAR_RX: track 36.3 -> 35.5 mm, vias 1 -> 0
- net +5V: track 332.2 -> 331.4 mm
- net GND: vias 16 -> 15

Commit message: Small optimisations and connected the final comp.
Routing:
- net PWM_R: track 316.3 -> 310.1 mm
- net +5V: track 331.4 -> 332.1 mm
- net GND: vias 15 -> 16
